File: zmote.kicad_pcb (KiCad board)
At the start: 2 copper layers, 50 x 50 mm, 88 parts, among them CON1 USB-MICRO-B, CON2 USB-MICRO-B, P1 CONN_01X01, P2 CONN_01X05, P3 CONN_01X05, P4 CONN_01X01, P5 CONN_01X01, Q2 BC547, U1 LD1117S33CTR, U3 ESP-01v090

Commit message: custom footprints
Parts:
- P3 (x4): footprint lib:Mounting5Holes_1mm -> zmote-custom:Mounting5Holes_1mm
- R1 (x4), R10 (x4), R2 (x4), R3 (x4), R4 (x4), R7 (x4), R8 (x4): footprint lib:Resistor_Horizontal_RM2.5mm -> zmote-custom:Resistor_Horizontal_RM2.5mm
